Commit message: Ready to use code

File: src/storm_description/urdf/storm_robot.urdf.xacro (robot description, xacro)
@@ -37,7 +37,4 @@
         <material name="grey"><color rgba="0.5 0.5 0.5 1"/></material>
       </visual>
-      <collision>
-        <geometry><box size="${robot_length} 0.10 ${robot_height}"/></geometry>
-      </collision>
       <inertial>
         <mass value="${tu_mass}"/>
@@ -96,4 +93,8 @@
       <axis xyz="0 1 0"/>
     </joint>
+  <gazebo reference="${prefix}_wheel">
+      <mu1>1.0</mu1>
+      <mu2>1.0</mu2>
+    </gazebo>
   </xacro:macro>
   <xacro:wheel prefix="fl" x="0.06"  y="0.08"/>
@@ -152,12 +153,12 @@
       <right_joint>fr_wheel_joint</right_joint>
       <right_joint>rr_wheel_joint</right_joint>
-      <wheel_separation>0.20</wheel_separation>
+      <wheel_separation>0.16</wheel_separation>
       <wheel_radius>0.05</wheel_radius>
-      <topic>cmd_vel</topic>
+      <topic>/model/storm/cmd_vel</topic>
     </plugin>
   </gazebo>
   <gazebo>
     <plugin filename="libignition-gazebo-joint-state-publisher-system.so" name="ignition::gazebo::systems::JointStatePublisher">
-      <topic>joint_states</topic>
+      <topic>/model/storm/joint_states</topic>
       <joint_name>vtm_joint</joint_name>
       <joint_name>fl_wheel_joint</joint_name>

Commit message: FIxed Lidar Latest Version

File: src/storm_description/urdf/storm_robot.urdf.xacro (robot description, xacro)
@@ -103,12 +103,15 @@
   <xacro:wheel prefix="rr" x="-0.06" y="-0.08"/>
   <!-- LIDAR Hokuyo -->
-  <joint name="lidar_joint" type="fixed">
+  <joint name="lidar_joint" type="revolute">
     <parent link="base_link"/>
     <child link="lidar_link"/>
     <origin xyz="0 0 0.10" rpy="0 0 0"/>
+    <axis xyz="0 0 1"/>
+    <!-- Limiti a zero per impedire che si muova realmente -->
+    <limit lower="0" upper="0" effort="0" velocity="0"/>
   </joint>
-  <gazebo reference="lidar_joint">
+  <!-- <gazebo reference="lidar_joint">
     <preserveFixedJoint>true</preserveFixedJoint>
-  </gazebo>
+  </gazebo> -->
   <link name="lidar_link">
     <visual>
@@ -116,7 +119,4 @@
       <material name="dark"><color rgba="0.2 0.2 0.2 1"/></material>
     </visual>
-    <collision>
-      <geometry><cylinder radius="0.03" length="0.05"/></geometry>
-    </collision>
     <inertial>
       <mass value="0.1"/>
@@ -124,26 +124,29 @@
     </inertial>
   </link>
-  <gazebo reference="lidar_link">
-    <sensor type="lidar" name="hokuyo_sensor">
-      <topic>scan</topic>
-      <ignition_frame_id>lidar_link</ignition_frame_id>
-      <update_rate>10</update_rate>
-      <ray>
-        <scan>
-          <horizontal>
-            <samples>512</samples>
-            <min_angle>-2.356</min_angle>
-            <max_angle>2.356</max_angle>
-          </horizontal>
-        </scan>
-        <range>
-          <min>0.15</min>
-          <max>5.00</max>
-        </range>
-      </ray>
-      <always_on>1</always_on>
-      <visualize>false</visualize>
-    </sensor>
-  </gazebo>
+ <gazebo reference="lidar_link">
+  <sensor name="hokuyo_sensor" type="gpu_lidar">
+    <pose>0 0 0 0 0 0</pose>
+    <topic>/model/storm/scan</topic>
+    <update_rate>10</update_rate>
+    <lidar>
+      <scan>
+        <horizontal>
+          <samples>512</samples>
+          <resolution>1</resolution>
+          <min_angle>-2.356</min_angle>
+          <max_angle>2.356</max_angle>
+        </horizontal>
+      </scan>
+      <range>
+        <min>0.15</min>
+        <max>5.0</max>
+        <resolution>0.01</resolution>
+      </range>
+      <visualize>true</visualize>
+    </lidar>
+    <always_on>true</always_on>
+    <ignition_frame_id>lidar_link</ignition_frame_id>
+  </sensor>
+</gazebo>
   <!-- Plugin DiffDrive per la locomozione -->
   <gazebo>
@@ -166,4 +169,6 @@
       <joint_name>rl_wheel_joint</joint_name>
       <joint_name>rr_wheel_joint</joint_name>
+      <joint_name>lidar_joint</joint_name>
+      <update_rate>30</update_rate>
     </plugin>
   </gazebo>

Commit message: codice funzionante

File: src/storm_description/urdf/storm_robot.urdf.xacro (robot description, xacro)
@@ -103,5 +103,5 @@
   <xacro:wheel prefix="rr" x="-0.06" y="-0.08"/>
   <!-- LIDAR Hokuyo -->
-  <joint name="lidar_joint" type="revolute">
+  <joint name="lidar_joint" type="fixed">
     <parent link="base_link"/>
     <child link="lidar_link"/>
@@ -125,5 +125,5 @@
   </link>
  <gazebo reference="lidar_link">
-  <sensor name="hokuyo_sensor" type="gpu_lidar">
+  <sensor name="lidar" type="gpu_lidar">
     <pose>0 0 0 0 0 0</pose>
     <topic>/model/storm/scan</topic>
@@ -169,6 +169,4 @@
       <joint_name>rl_wheel_joint</joint_name>
       <joint_name>rr_wheel_joint</joint_name>
-      <joint_name>lidar_joint</joint_name>
-      <update_rate>30</update_rate>
     </plugin>
   </gazebo>

Commit message: latest code on 15 May

File: src/storm_description/urdf/storm_robot.urdf.xacro (robot description, xacro)
@@ -2,8 +2,7 @@
 <robot xmlns:xacro="http://www.ros.org/wiki/xacro" name="storm_robot">
   <!-- Proprietà fisiche STORM -->
-  <xacro:property name="tu_mass"     value="2.81"/>
-  <xacro:property name="wu_mass"     value="0.76"/>
-  <xacro:property name="vtu_mass"    value="0.73"/>
-  <xacro:property name="base_mass"   value="1.26"/>
+  <xacro:property name="tu_mass"      value="2.81"/>
+  <xacro:property name="wu_mass"      value="0.76"/>
+  <xacro:property name="base_mass"    value="1.26"/>
   <xacro:property name="robot_length" value="0.410"/>
   <xacro:property name="robot_width"  value="0.305"/>
@@ -50,25 +49,7 @@
   <xacro:tracked_unit prefix="left"  y="0.1025"/>
   <xacro:tracked_unit prefix="right" y="-0.1025"/>
-  <!-- Meccanismo di Traslazione Verticale (VTM) -->
-  <joint name="vtm_joint" type="prismatic">
-    <parent link="base_link"/>
-    <child link="vtu_link"/>
-    <axis xyz="0 0 -1"/>
-    <limit lower="0" upper="0.05" effort="1000" velocity="0.1"/>
-  </joint>
-  <link name="vtu_link">
-    <visual>
-      <geometry><box size="0.15 0.15 0.04"/></geometry>
-      <material name="black"><color rgba="0.1 0.1 0.1 1"/></material>
-    </visual>
-    <collision>
-      <geometry><box size="0.15 0.15 0.04"/></geometry>
-    </collision>
-    <inertial>
-      <mass value="${vtu_mass}"/>
-      <inertia ixx="0.001" iyy="0.001" izz="0.001" ixy="0" ixz="0" iyz="0"/>
-    </inertial>
-  </link>
   <!-- Macro per Unità a Ruote (Wheeled Units) -->
+  <!-- VTM rimosso: ruote collegate direttamente a base_link -->
+  <!-- Questo elimina il joint prismatico che causava instabilità del solver -->
   <xacro:macro name="wheel" params="prefix x y">
     <link name="${prefix}_wheel">
@@ -76,5 +57,5 @@
         <origin rpy="1.5708 0 0"/>
         <geometry><cylinder radius="0.05" length="0.04"/></geometry>
-        <material name="black"/>
+        <material name="black"><color rgba="0.1 0.1 0.1 1"/></material>
       </visual>
       <collision>
@@ -88,10 +69,10 @@
     </link>
     <joint name="${prefix}_wheel_joint" type="continuous">
-      <parent link="vtu_link"/>
+      <parent link="base_link"/>
       <child link="${prefix}_wheel"/>
       <origin xyz="${x} ${y} -0.04"/>
       <axis xyz="0 1 0"/>
     </joint>
-  <gazebo reference="${prefix}_wheel">
+    <gazebo reference="${prefix}_wheel">
       <mu1>1.0</mu1>
       <mu2>1.0</mu2>
@@ -107,11 +88,5 @@
     <child link="lidar_link"/>
     <origin xyz="0 0 0.10" rpy="0 0 0"/>
-    <axis xyz="0 0 1"/>
-    <!-- Limiti a zero per impedire che si muova realmente -->
-    <limit lower="0" upper="0" effort="0" velocity="0"/>
   </joint>
-  <!-- <gazebo reference="lidar_joint">
-    <preserveFixedJoint>true</preserveFixedJoint>
-  </gazebo> -->
   <link name="lidar_link">
     <visual>
@@ -124,29 +99,29 @@
     </inertial>
   </link>
- <gazebo reference="lidar_link">
-  <sensor name="lidar" type="gpu_lidar">
-    <pose>0 0 0 0 0 0</pose>
-    <topic>/model/storm/scan</topic>
-    <update_rate>10</update_rate>
-    <lidar>
-      <scan>
-        <horizontal>
-          <samples>512</samples>
-          <resolution>1</resolution>
-          <min_angle>-2.356</min_angle>
-          <max_angle>2.356</max_angle>
-        </horizontal>
-      </scan>
-      <range>
-        <min>0.15</min>
-        <max>5.0</max>
-        <resolution>0.01</resolution>
-      </range>
-      <visualize>true</visualize>
-    </lidar>
-    <always_on>true</always_on>
-    <ignition_frame_id>lidar_link</ignition_frame_id>
-  </sensor>
-</gazebo>
+  <gazebo reference="lidar_link">
+    <sensor name="lidar" type="gpu_lidar">
+      <pose>0 0 0 0 0 0</pose>
+      <topic>/model/storm/scan</topic>
+      <update_rate>10</update_rate>
+      <lidar>
+        <scan>
+          <horizontal>
+            <samples>512</samples>
+            <resolution>1</resolution>
+            <min_angle>-2.356</min_angle>
+            <max_angle>2.356</max_angle>
+          </horizontal>
+        </scan>
+        <range>
+          <min>0.15</min>
+          <max>5.0</max>
+          <resolution>0.01</resolution>
+        </range>
+        <visualize>true</visualize>
+      </lidar>
+      <always_on>true</always_on>
+      <ignition_frame_id>lidar_link</ignition_frame_id>
+    </sensor>
+  </gazebo>
   <!-- Plugin DiffDrive per la locomozione -->
   <gazebo>
@@ -164,5 +139,4 @@
     <plugin filename="libignition-gazebo-joint-state-publisher-system.so" name="ignition::gazebo::systems::JointStatePublisher">
       <topic>/model/storm/joint_states</topic>
-      <joint_name>vtm_joint</joint_name>
       <joint_name>fl_wheel_joint</joint_name>
       <joint_name>fr_wheel_joint</joint_name>
